Commit message: feat (hi2_update): update hi2 urdf and training config

File: assets/robots/ZJ-Humanoid/hi2/21dof/hi2_21dof.urdf (robot description, URDF)
Before this commit: robot hi, 30 links, 29 joints
Links:
- link left_shoulder_pitch_link: geometry visual mesh filename=../meshes/SCAPULA_L.STL
- link left_shoulder_roll_link: geometry visual mesh filename=../meshes/SHOULDER_L.STL
- link right_shoulder_pitch_link: geometry visual mesh filename=../meshes/SCAPULA_R.STL
- link right_shoulder_roll_link: geometry visual mesh filename=../meshes/SHOULDER_R.STL
